Commit message: map

File: description/robot.urdf (robot description, URDF)
Before this commit: robot my_bot, 5 links, 4 joints
Links:
- removed link world
- added link map
Joints:
- joint x_joint: parent world -> map

Commit message: simplified maps

File: description/robot.urdf (robot description, URDF)
Before this commit: robot my_bot, 5 links, 4 joints
Links:
- removed link map
- added link world
Joints:
- joint x_joint: parent map -> world
